Commit message: one leg

File: robot.urdf (robot description, URDF)
Before this commit: robot my_robot, 6 links, 6 joints
Links:
- removed link swing_leg
Joints:
- removed joint hip_pin

Commit message: longer leg

File: robot.urdf (robot description, URDF)
Before this commit: robot my_robot, 6 links, 6 joints
Links:
- link stance_leg: geometry visual cylinder length=1.2 radius=.01; visual sphere radius=.05

Commit message: heavy body

File: robot.urdf (robot description, URDF)
Before this commit: robot my_robot, 6 links, 6 joints
Links:
- link body: mass 1 -> 5
